File: sbc-exp-control/sbc-exp-control.kicad_sch (KiCad schematic)
At the start: 15 parts, among them J1 SBC_EXP, SW1 SW_Push, SW2 SW_Push, SW3 SW_Push, SW4 SW_Push, SW5 SW_Push, SW6 SW_Push, SW7 SW_Push

Commit message: SBC v2.3
Fixes over v2.2:

  - SBC: Fix the VIA footprint: CA1 and CB1 are inputs
  - SBC: Move the microSD power enable line from (VIA3) CA1 (input) to CA2 (output)
  - Controller: connect LED enable
  - Controller: SMT switches
Parts:
- SW1, SW2, SW3, SW4, SW5, SW6, SW7: footprint Button_Switch_THT:SW_PUSH_6mm -> Button_Switch_SMD:SW_Push_1P1T_NO_6x6mm_H9.5mm
Changed lines of the file:
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@@
   (title_block
     (title "6502 SBC Expansion - Controller")
-    (date "2022-03-07")
-    (rev "2.2")
+    (date "2022-06-14")
+    (rev "2.3")
   )
   (junction (at 172.72 71.755) (diameter 0) (color 0 0 0 0)
@@
     (property "Reference" "SW5" (id 0) (at 200.66 57.785 0))
     (property "Value" "SW_Push" (id 1) (at 200.66 60.325 0))
-    (property "Footprint" "Button_Switch_THT:SW_PUSH_6mm" (id 2) (at 200.66 60.325 0)
+    (property "Footprint" "Button_Switch_SMD:SW_Push_1P1T_NO_6x6mm_H9.5mm" (id 2) (at 200.66 60.325 0)
       (effects (font (size 1.27 1.27)) hide)
     )
@@
     (property "Reference" "SW6" (id 0) (at 217.17 57.785 0))
     (property "Value" "SW_Push" (id 1) (at 217.17 60.325 0))
-    (property "Footprint" "Button_Switch_THT:SW_PUSH_6mm" (id 2) (at 217.17 60.325 0)
+    (property "Footprint" "Button_Switch_SMD:SW_Push_1P1T_NO_6x6mm_H9.5mm" (id 2) (at 217.17 60.325 0)
       (effects (font (size 1.27 1.27)) hide)
     )
@@
     (property "Reference" "SW7" (id 0) (at 233.68 57.785 0))
     (property "Value" "SW_Push" (id 1) (at 233.68 60.325 0))
-    (property "Footprint" "Button_Switch_THT:SW_PUSH_6mm" (id 2) (at 233.68 60.325 0)
+    (property "Footprint" "Button_Switch_SMD:SW_Push_1P1T_NO_6x6mm_H9.5mm" (id 2) (at 233.68 60.325 0)
       (effects (font (size 1.27 1.27)) hide)
     )
@@
     (property "Reference" "SW4" (id 0) (at 184.15 57.785 0))
     (property "Value" "SW_Push" (id 1) (at 184.15 60.325 0))
-    (property "Footprint" "Button_Switch_THT:SW_PUSH_6mm" (id 2) (at 184.15 60.325 0)
+    (property "Footprint" "Button_Switch_SMD:SW_Push_1P1T_NO_6x6mm_H9.5mm" (id 2) (at 184.15 60.325 0)
       (effects (font (size 1.27 1.27)) hide)
     )
@@
     (property "Reference" "SW1" (id 0) (at 134.62 57.785 0))
     (property "Value" "SW_Push" (id 1) (at 134.62 60.325 0))
-    (property "Footprint" "Button_Switch_THT:SW_PUSH_6mm" (id 2) (at 134.62 60.325 0)
+    (property "Footprint" "Button_Switch_SMD:SW_Push_1P1T_NO_6x6mm_H9.5mm" (id 2) (at 134.62 60.325 0)
       (effects (font (size 1.27 1.27)) hide)
     )
@@
     (property "Reference" "SW3" (id 0) (at 167.64 57.785 0))
     (property "Value" "SW_Push" (id 1) (at 167.64 60.325 0))
-    (property "Footprint" "Button_Switch_THT:SW_PUSH_6mm" (id 2) (at 167.64 60.325 0)
+    (property "Footprint" "Button_Switch_SMD:SW_Push_1P1T_NO_6x6mm_H9.5mm" (id 2) (at 167.64 60.325 0)
       (effects (font (size 1.27 1.27)) hide)
     )
@@
     (property "Reference" "SW2" (id 0) (at 151.13 57.785 0))
     (property "Value" "SW_Push" (id 1) (at 151.13 60.325 0))
-    (property "Footprint" "Button_Switch_THT:SW_PUSH_6mm" (id 2) (at 151.13 60.325 0)
+    (property "Footprint" "Button_Switch_SMD:SW_Push_1P1T_NO_6x6mm_H9.5mm" (id 2) (at 151.13 60.325 0)
       (effects (font (size 1.27 1.27)) hide)
     )
@@
     )
     (path "/5b6b1e39-f691-4099-abbb-198bb062b2a5"
-      (reference "SW1") (unit 1) (value "SW_Push") (footprint "Button_Switch_THT:SW_PUSH_6mm")
+      (reference "SW1") (unit 1) (value "SW_Push") (footprint "Button_Switch_SMD:SW_Push_1P1T_NO_6x6mm_H9.5mm")
     )
     (path "/e7df1f41-fb84-4e8a-8fb4-7075427d7230"
-      (reference "SW2") (unit 1) (value "SW_Push") (footprint "Button_Switch_THT:SW_PUSH_6mm")
+      (reference "SW2") (unit 1) (value "SW_Push") (footprint "Button_Switch_SMD:SW_Push_1P1T_NO_6x6mm_H9.5mm")
     )
     (path "/97c6714b-e883-4340-befa-4143b261248f"
-      (reference "SW3") (unit 1) (value "SW_Push") (footprint "Button_Switch_THT:SW_PUSH_6mm")
+      (reference "SW3") (unit 1) (value "SW_Push") (footprint "Button_Switch_SMD:SW_Push_1P1T_NO_6x6mm_H9.5mm")
     )
     (path "/5aeac1bd-a36c-4926-b80f-558014ee5ac7"
-      (reference "SW4") (unit 1) (value "SW_Push") (footprint "Button_Switch_THT:SW_PUSH_6mm")
+      (reference "SW4") (unit 1) (value "SW_Push") (footprint "Button_Switch_SMD:SW_Push_1P1T_NO_6x6mm_H9.5mm")
     )
     (path "/16d0b933-f9f7-4b03-8e78-9b4312677781"
-      (reference "SW5") (unit 1) (value "SW_Push") (footprint "Button_Switch_THT:SW_PUSH_6mm")
+      (reference "SW5") (unit 1) (value "SW_Push") (footprint "Button_Switch_SMD:SW_Push_1P1T_NO_6x6mm_H9.5mm")
     )
     (path "/343428f4-484a-4340-bd70-3fec20ff1ed0"
-      (reference "SW6") (unit 1) (value "SW_Push") (footprint "Button_Switch_THT:SW_PUSH_6mm")
+      (reference "SW6") (unit 1) (value "SW_Push") (footprint "Button_Switch_SMD:SW_Push_1P1T_NO_6x6mm_H9.5mm")
     )
     (path "/35825b93-e118-4eca-88c2-dcef148bebc1"
-      (reference "SW7") (unit 1) (value "SW_Push") (footprint "Button_Switch_THT:SW_PUSH_6mm")
-    )
-  )
+      (reference "SW7") (unit 1) (value "SW_Push") (footprint "Button_Switch_SMD:SW_Push_1P1T_NO_6x6mm_H9.5mm")
+    )
+  )
