File: sbc/sbc-via.kicad_sch (KiCad schematic)
At the start: 10 parts, among them J1 EXP_1A, J2 EXP_1B, J3 EXP_2A, J4 EXP_2B, U7 WD65C22, U8 WD65C22, U9 WD65C22

Commit message: SBC v2.3
Fixes over v2.2:

  - SBC: Fix the VIA footprint: CA1 and CB1 are inputs
  - SBC: Move the microSD power enable line from (VIA3) CA1 (input) to CA2 (output)
  - SBC: Tie 65C02 SOB high
  - Controller: connect LED enable
  - Controller: SMT switches
Connections:
- net SD_PWR: now also U9.39 (CA2); no longer U9.40 (CA1)
Changed lines of the file:
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@@
   (title_block
     (title "6502 SBC")
-    (date "2022-03-07")
-    (rev "2.2")
+    (date "2023-02-07")
+    (rev "2.3")
   )
   (junction (at 53.34 20.32) (diameter 0) (color 0 0 0 0)
@@
   (junction (at 215.9 121.92) (diameter 0) (color 0 0 0 0)
   )
-  (no_connect (at 237.49 53.34))
+  (no_connect (at 237.49 50.8))
   (no_connect (at 140.97 182.88))
   (no_connect (at 59.69 144.78))
@@
     )
   )
-  (global_label "VIA1_CA1" (shape bidirectional) (at 74.93 50.8 0) (fields_autoplaced)
+  (global_label "VIA1_CA1" (shape input) (at 74.93 50.8 0) (fields_autoplaced)
     (effects (font (size 1.27 1.27)) (justify left))
     (property "Intersheet References" "${INTERSHEET_REFS}" (id 0) (at 85.8702 50.7206 0)
@@
     )
   )
-  (global_label "VIA2_CA1" (shape bidirectional) (at 156.21 50.8 0) (fields_autoplaced)
+  (global_label "VIA2_CA1" (shape input) (at 156.21 50.8 0) (fields_autoplaced)
     (effects (font (size 1.27 1.27)) (justify left))
     (property "Intersheet References" "${INTERSHEET_REFS}" (id 0) (at 167.1502 50.7206 0)
@@
     )
   )
-  (global_label "VIA2_CA1" (shape bidirectional) (at 128.27 129.54 180) (fields_autoplaced)
-    (effects (font (size 1.27 1.27)) (justify right))
-    (property "Intersheet References" "${INTERSHEET_REFS}" (id 0) (at 117.3298 129.6194 0)
+  (global_label "VIA2_CA1" (shape output) (at 128.27 129.54 180) (fields_autoplaced)
+    (effects (font (size 1.27 1.27)) (justify right))
+    (property "Intersheet References" "${INTERSHEET_REFS}" (id 0) (at 117.3298 129.4606 0)
       (effects (font (size 1.27 1.27)) (justify right) hide)
     )
@@
     )
   )
-  (global_label "SD_PWR" (shape output) (at 237.49 50.8 0) (fields_autoplaced)
-    (effects (font (size 1.27 1.27)) (justify left))
-    (property "Intersheet References" "${INTERSHEET_REFS}" (id 0) (at 247.3417 50.8794 0)
+  (global_label "SD_PWR" (shape output) (at 237.49 53.34 0) (fields_autoplaced)
+    (effects (font (size 1.27 1.27)) (justify left))
+    (property "Intersheet References" "${INTERSHEET_REFS}" (id 0) (at 247.3417 53.4194 0)
       (effects (font (size 1.27 1.27)) (justify left) hide)
     )
@@
     )
   )
-  (global_label "VIA2_CB1" (shape bidirectional) (at 156.21 83.82 0) (fields_autoplaced)
+  (global_label "VIA2_CB1" (shape input) (at 156.21 83.82 0) (fields_autoplaced)
     (effects (font (size 1.27 1.27)) (justify left))
     (property "Intersheet References" "${INTERSHEET_REFS}" (id 0) (at 167.3317 83.7406 0)
@@
     )
   )
-  (global_label "VIA1_CB1" (shape bidirectional) (at 74.93 83.82 0) (fields_autoplaced)
+  (global_label "VIA1_CB1" (shape input) (at 74.93 83.82 0) (fields_autoplaced)
     (effects (font (size 1.27 1.27)) (justify left))
     (property "Intersheet References" "${INTERSHEET_REFS}" (id 0) (at 86.0517 83.7406 0)
@@
     )
   )
-  (global_label "VIA2_CB1" (shape bidirectional) (at 128.27 177.8 180) (fields_autoplaced)
+  (global_label "VIA2_CB1" (shape output) (at 128.27 177.8 180) (fields_autoplaced)
     (effects (font (size 1.27 1.27)) (justify right))
     (property "Intersheet References" "${INTERSHEET_REFS}" (id 0) (at 117.1483 177.7206 0)
@@
     )
   )
-  (global_label "VIA1_CA1" (shape bidirectional) (at 59.69 134.62 180) (fields_autoplaced)
-    (effects (font (size 1.27 1.27)) (justify right))
-    (property "Intersheet References" "${INTERSHEET_REFS}" (id 0) (at 48.7498 134.6994 0)
+  (global_label "VIA1_CA1" (shape output) (at 59.69 134.62 180) (fields_autoplaced)
+    (effects (font (size 1.27 1.27)) (justify right))
+    (property "Intersheet References" "${INTERSHEET_REFS}" (id 0) (at 48.7498 134.5406 0)
       (effects (font (size 1.27 1.27)) (justify right) hide)
     )
@@
     )
   )
-  (global_label "VIA1_CB1" (shape bidirectional) (at 59.69 182.88 180) (fields_autoplaced)
-    (effects (font (size 1.27 1.27)) (justify right))
-    (property "Intersheet References" "${INTERSHEET_REFS}" (id 0) (at 48.5683 182.9594 0)
-      (effects (font (size 1.27 1.27)) (justify right) hide)
-    )
+  (global_label "VIA1_CB1" (shape output) (at 59.69 182.88 180) (fields_autoplaced)
+    (effects (font (size 1.27 1.27)) (justify right))
+    (property "Intersheet References" "${INTERSHEET_REFS}" (id 0) (at 48.5683 182.8006 0)
+      (effects (font (size 1.27 1.27)) (justify right) hide)
+    )
